Commit message: integrate with pineapple v2 controller

File: controller/robot/pineapple_v2/urdf/pineappleV2.urdf (robot description, URDF)
Before this commit: robot pineapple_v2, 18 links, 17 joints
Links:
- link L_calf: geometry collision box size=0.052 0.021 0.122; collision cylinder length=0.021 radius=0.026
- link L_hip: geometry visual mesh filename=../meshes/L_hip.STL
- link L_thigh: geometry collision box size=0.056 0.028 0.11; collision cylinder length=0.028 radius=0.028
- link L_wheel: geometry collision cylinder length=0.007 radius=0.077; visual mesh filename=../meshes/L_wheel.STL
- link R_calf: geometry collision box size=0.052 0.021 0.122; collision cylinder length=0.021 radius=0.026
- link R_hip: geometry visual mesh filename=../meshes/R_hip.STL
- link R_thigh: geometry collision box size=0.056 0.028 0.11; collision cylinder length=0.028 radius=0.028
- link R_wheel: geometry collision cylinder length=0.007 radius=0.077; visual mesh filename=../meshes/R_wheel.STL
- link arm_base: geometry visual mesh filename=../meshes/arm_base.STL
- link base_link: geometry collision box size=0.31 0.15 0.13; visual mesh filename=../meshes/base_link.STL
- link battery: geometry visual mesh filename=../meshes/battery.STL
- link camera: geometry visual mesh filename=../meshes/camera.STL
- link hip_motor_L: geometry visual mesh filename=../meshes/hip_motor_L.STL
- link hip_motor_R: geometry visual mesh filename=../meshes/hip_motor_R.STL
- link knee_motor_L: geometry visual mesh filename=../meshes/knee_motor_L.STL
- link knee_motor_R: geometry visual mesh filename=../meshes/knee_motor_R.STL
- link wheel_motor_L: geometry visual mesh filename=../meshes/wheel_motor_L.STL
- link wheel_motor_R: geometry visual mesh filename=../meshes/wheel_motor_R.STL
